Commit message: Spawn robot (URDF v1) in home_sim.launch.py
- launch: robot_state_publisher (use_sim_time) + spawn_entity.py from
  /robot_description; args spawn_robot, x, y, z, yaw (default = S1 in
  config/trials.yaml); prepend share/ parent to GAZEBO_MODEL_PATH so
  package:// meshes (converted to model:// by sdformat) resolve.
- CMakeLists: install urdf/ and meshes/.
- package.xml: exec_depend launch_ros, robot_state_publisher, xacro.
- URDF v1: mesh URIs -> package://objectnav_sim_gazebo; collision uses
  primitives measured from the meshes (4 chassis boxes with a gap at the
  LiDAR scan plane, wheel cylinders) instead of ~1e5-triangle STLs;
  wheel inertia about the spin axis (y) = 1/2 m r^2; Gazebo materials;
  zero friction on the fixed caster.

Co-Authored-By: Claude Opus 5.5 <noreply@anthropic.com>
Claude-Session: https://claude.ai/code/session_01Jj5wz3bwKX9mzVkh9HTVm8

File: urdf/mobile_robot.urdf.xacro (robot description, xacro)
@@ -1,4 +1,8 @@
 <?xml version="1.0"?>
 <robot xmlns:xacro="http://www.ros.org/wiki/xacro" name="mobile_robot">
+    <!-- Robot mô phỏng = URDF v1 của receptionist_robot (urdf/mobile_robot.urdf.xacro, mesh Model_v1.stl).
+         Mesh trỏ vào chính gói này (package://objectnav_sim_gazebo/meshes/...). Khi URDF -> SDF, sdformat đổi
+         package:// thành model://, nên home_sim.launch.py thêm thư mục share/ của gói vào GAZEBO_MODEL_PATH.
+         Collision dùng hình khối đơn giản (đo từ mesh) thay cho mesh STL ~1e5 tam giác. -->
     <!-- ==================== MATERIALS & MACROS ==================== -->
     <material name="white">
@@ -32,4 +36,14 @@
         </inertial>
     </xacro:macro>
+    <!-- Trụ đặc có trục đối xứng theo y (trục quay của bánh: joint axis = 0 1 0) -> iyy = 1/2 m r^2 -->
+    <xacro:macro name="inertial_cylinder_y" params="mass length radius *origin">
+        <inertial>
+            <xacro:insert_block name="origin"/>
+            <mass value="${mass}" />
+            <inertia ixx="${(1/12) * mass * (3*radius*radius + length*length)}" ixy="0.0" ixz="0.0"
+                     iyy="${(1/2) * mass * (radius*radius)}" iyz="0.0"
+                     izz="${(1/12) * mass * (3*radius*radius + length*length)}" />
+        </inertial>
+    </xacro:macro>
     <xacro:macro name="inertial_sphere" params="mass radius *origin">
         <inertial>
@@ -76,14 +90,28 @@
             <origin xyz="0 0 0" rpy="0 0 0"/>
             <geometry>
-                <mesh filename="package://mobile_robot/meshes/Model_v1.stl" scale="0.001 0.001 0.001"/>
+                <mesh filename="package://objectnav_sim_gazebo/meshes/Model_v1.stl" scale="0.001 0.001 0.001"/>
             </geometry>
             <material name="white"/>
         </visual>
-        <collision>
-            <!-- <origin xyz="0.03 0 0.05" rpy="0 0 0"/> -->
-            <origin xyz="0 0 0" rpy="0 0 0"/>
-            <geometry>
-                <mesh filename="package://mobile_robot/meshes/Model_v1.stl" scale="0.001 0.001 0.001"/>
-            </geometry>
+        <!-- Collision: 4 hộp bao theo lát cắt chiều cao của Model_v1.stl (khung base_link, m):
+             thân dưới x[-0.100,0.292] y[±0.201] z[-0.011,0.530]; cột x[-0.030,0.222] y[±0.126] z[0.530,1.130];
+             đầu x[-0.030,0.291] y[±0.178] z[1.130,1.373].
+             Chừa khe z[0.045,0.110] quanh mặt quét LiDAR (laser_frame z=0.085, mesh RPLiDAR z[0.058,0.097])
+             để cảm biến ray (khi thêm sau) không bị chính thân robot che. -->
+        <collision name="chassis_base_low">
+            <origin xyz="0.096 0 0.017" rpy="0 0 0"/>
+            <geometry><box size="0.392 0.402 0.056"/></geometry>
+        </collision>
+        <collision name="chassis_base_high">
+            <origin xyz="0.096 0 0.320" rpy="0 0 0"/>
+            <geometry><box size="0.392 0.402 0.420"/></geometry>
+        </collision>
+        <collision name="chassis_column">
+            <origin xyz="0.096 0 0.830" rpy="0 0 0"/>
+            <geometry><box size="0.252 0.252 0.600"/></geometry>
+        </collision>
+        <collision name="chassis_head">
+            <origin xyz="0.1305 0 1.2515" rpy="0 0 0"/>
+            <geometry><box size="0.321 0.356 0.243"/></geometry>
         </collision>
         <xacro:inertial_box mass="${chassis_mass}" x="${chassis_length}" y="${chassis_width}" z="${chassis_height}">
@@ -101,17 +129,18 @@
             <origin xyz="0 0 0" rpy="0 0 0"/>
             <geometry>
-                <mesh filename="package://mobile_robot/meshes/hoverboard_motor_assembly.stl" scale="0.001 0.001 0.001"/>
+                <mesh filename="package://objectnav_sim_gazebo/meshes/hoverboard_motor_assembly.stl" scale="0.001 0.001 0.001"/>
             </geometry>
             <material name="blue"/>
         </visual>
-        <collision>
-            <origin xyz="0 0 0" rpy="0 0 0"/>
-            <geometry>
-                <mesh filename="package://mobile_robot/meshes/hoverboard_motor_assembly.stl" scale="0.001 0.001 0.001"/>
-            </geometry>
-        </collision>
-        <xacro:inertial_cylinder mass="${wheel_mass}" length="${wheel_width}" radius="${wheel_radius}">
-            <origin xyz="0 0 0" rpy="0 0 0"/>
-        </xacro:inertial_cylinder>
+        <!-- Collision: trụ bán kính wheel_radius, trục theo y (lốp nằm ở y∈[-0.02,0.02] của mesh) -->
+        <collision>
+            <origin xyz="0 0 0" rpy="${pi/2} 0 0"/>
+            <geometry>
+                <cylinder radius="${wheel_radius}" length="${wheel_width}"/>
+            </geometry>
+        </collision>
+        <xacro:inertial_cylinder_y mass="${wheel_mass}" length="${wheel_width}" radius="${wheel_radius}">
+            <origin xyz="0 0 0" rpy="0 0 0"/>
+        </xacro:inertial_cylinder_y>
     </link>
     <joint name="right_wheel_joint" type="continuous">
@@ -125,17 +154,18 @@
             <origin xyz="0 0 0" rpy="0 0 0"/>
             <geometry>
-                <mesh filename="package://mobile_robot/meshes/hoverboard_motor_assembly.stl" scale="0.001 0.001 0.001"/>
+                <mesh filename="package://objectnav_sim_gazebo/meshes/hoverboard_motor_assembly.stl" scale="0.001 0.001 0.001"/>
             </geometry>
             <material name="blue"/>
         </visual>
-        <collision>
-            <origin xyz="0 0 0" rpy="0 0 0"/>
-            <geometry>
-                <mesh filename="package://mobile_robot/meshes/hoverboard_motor_assembly.stl" scale="0.001 0.001 0.001"/>
-            </geometry>
-        </collision>
-        <xacro:inertial_cylinder mass="${wheel_mass}" length="${wheel_width}" radius="${wheel_radius}">
-            <origin xyz="0 0 0" rpy="0 0 0"/>
-        </xacro:inertial_cylinder>
+        <!-- Collision: trụ bán kính wheel_radius, trục theo y (lốp nằm ở y∈[-0.02,0.02] của mesh) -->
+        <collision>
+            <origin xyz="0 0 0" rpy="${pi/2} 0 0"/>
+            <geometry>
+                <cylinder radius="${wheel_radius}" length="${wheel_width}"/>
+            </geometry>
+        </collision>
+        <xacro:inertial_cylinder_y mass="${wheel_mass}" length="${wheel_width}" radius="${wheel_radius}">
+            <origin xyz="0 0 0" rpy="0 0 0"/>
+        </xacro:inertial_cylinder_y>
     </link>
     <joint name="caster_wheel_joint" type="fixed">
@@ -148,5 +178,5 @@
             <origin xyz="0 0 0" rpy="0 0 0"/>
             <geometry>
-                <mesh filename="package://mobile_robot/meshes/caster_wheel.stl" scale="0.01 0.01 0.01"/>
+                <mesh filename="package://objectnav_sim_gazebo/meshes/caster_wheel.stl" scale="0.01 0.01 0.01"/>
             </geometry>
             <material name="black"/>
@@ -172,5 +202,5 @@
             <geometry>
                 <!-- <cylinder length="0.04" radius="0.038"/> -->
-                <mesh filename="package://mobile_robot/meshes/RPLiDAR_s2.stl" scale="0.001 0.001 0.001"/>
+                <mesh filename="package://objectnav_sim_gazebo/meshes/RPLiDAR_s2.stl" scale="0.001 0.001 0.001"/>
             </geometry>
             <material name="black"/>
@@ -180,5 +210,5 @@
             <geometry>
                 <cylinder length="0.04" radius="0.038"/>
-                <!-- <mesh filename="package://mobile_robot/meshes/RPLiDAR_s2.stl" scale="0.001 0.001 0.001"/> -->
+                <!-- <mesh filename="package://objectnav_sim_gazebo/meshes/RPLiDAR_s2.stl" scale="0.001 0.001 0.001"/> -->
             </geometry>
         </collision>
@@ -220,4 +250,5 @@
             </xacro:inertial_box>
         </link>
+        <gazebo reference="${name}_link"><material>Gazebo/Blue</material></gazebo>
     </xacro:macro>
     <!-- TOP -->
@@ -273,3 +304,16 @@
     </joint>
     <xacro:ultrasonic_link name="us_bot_right"/> -->
+    <!-- ==================== GAZEBO ==================== -->
+    <!-- sdformat (sdf9) không chuyển <material><color> của URDF sang SDF, nên đặt màu Gazebo riêng -->
+    <gazebo reference="chassis"><material>Gazebo/White</material></gazebo>
+    <gazebo reference="left_wheel"><material>Gazebo/Blue</material></gazebo>
+    <gazebo reference="right_wheel"><material>Gazebo/Blue</material></gazebo>
+    <gazebo reference="laser_frame"><material>Gazebo/Black</material></gazebo>
+    <gazebo reference="imu_link"><material>Gazebo/Blue</material></gazebo>
+    <!-- Bánh caster gắn cứng (fixed joint) -> ma sát 0 để nó trượt thay vì lăn -->
+    <gazebo reference="caster_wheel">
+        <material>Gazebo/Black</material>
+        <mu1>0.0</mu1>
+        <mu2>0.0</mu2>
+    </gazebo>
 </robot>

Commit message: Add diff-drive, 2D LiDAR, IMU plugins; load meshes via file://
- Mesh URIs come from xacro arg mesh_uri; the launch passes
  file://<share>/meshes (Gazebo 11 SystemPaths::FindFileURI reads absolute
  paths), so share/ is no longer added to GAZEBO_MODEL_PATH and gzclient's
  "Missing model.config" errors go away. Default stays package:// for RViz.
- libgazebo_ros_diff_drive: /cmd_vel -> wheels, /odom from encoders,
  separation 0.464 m, diameter 0.168 m (= wheel_odom_params.yaml),
  publish_odom_tf configurable (false when running EKF).
- Right wheel joint axis 0 -1 0: with the joint frame yawed by pi this is
  +y in base_link, so positive velocity drives forward on both wheels as
  gazebo_ros_diff_drive assumes.
- libgazebo_ros_ray_sensor on laser_frame: RPLIDAR S2 spec (0.05-30 m,
  10 Hz, 0.1125 deg = 3200 samples), /scan; samples configurable.
- libgazebo_ros_imu_sensor on imu_link: /imu/data, 100 Hz.
- libgazebo_ros_joint_state_publisher for both wheels.
- launch: robot_description built in OpaqueFunction from launch args
  publish_odom_tf and lidar_samples.

Co-Authored-By: Claude Opus 5.5 <noreply@anthropic.com>
Claude-Session: https://claude.ai/code/session_01Jj5wz3bwKX9mzVkh9HTVm8

File: urdf/mobile_robot.urdf.xacro (robot description, xacro)
@@ -2,7 +2,12 @@
 <robot xmlns:xacro="http://www.ros.org/wiki/xacro" name="mobile_robot">
     <!-- Robot mô phỏng = URDF v1 của receptionist_robot (urdf/mobile_robot.urdf.xacro, mesh Model_v1.stl).
-         Mesh trỏ vào chính gói này (package://objectnav_sim_gazebo/meshes/...). Khi URDF -> SDF, sdformat đổi
-         package:// thành model://, nên home_sim.launch.py thêm thư mục share/ của gói vào GAZEBO_MODEL_PATH.
+         mesh_uri: home_sim.launch.py truyền file://<share>/meshes (Gazebo 11 đọc trực tiếp đường dẫn tuyệt đối,
+         không cần GAZEBO_MODEL_PATH); mặc định package:// dùng cho RViz / xacro chạy tay.
          Collision dùng hình khối đơn giản (đo từ mesh) thay cho mesh STL ~1e5 tam giác. -->
+    <xacro:arg name="mesh_uri" default="package://objectnav_sim_gazebo/meshes"/>
+    <xacro:arg name="publish_odom_tf" default="true"/>
+    <xacro:arg name="lidar_samples" default="3200"/>
+    <xacro:property name="mesh_uri" value="$(arg mesh_uri)"/>
+    <xacro:property name="lidar_samples" value="$(arg lidar_samples)"/>
     <!-- ==================== MATERIALS & MACROS ==================== -->
     <material name="white">
@@ -90,5 +95,5 @@
             <origin xyz="0 0 0" rpy="0 0 0"/>
             <geometry>
-                <mesh filename="package://objectnav_sim_gazebo/meshes/Model_v1.stl" scale="0.001 0.001 0.001"/>
+                <mesh filename="${mesh_uri}/Model_v1.stl" scale="0.001 0.001 0.001"/>
             </geometry>
             <material name="white"/>
@@ -129,5 +134,5 @@
             <origin xyz="0 0 0" rpy="0 0 0"/>
             <geometry>
-                <mesh filename="package://objectnav_sim_gazebo/meshes/hoverboard_motor_assembly.stl" scale="0.001 0.001 0.001"/>
+                <mesh filename="${mesh_uri}/hoverboard_motor_assembly.stl" scale="0.001 0.001 0.001"/>
             </geometry>
             <material name="blue"/>
@@ -148,5 +153,8 @@
         <child link="right_wheel"/>
         <origin xyz="0 -${wheel_offset_y} 0" rpy="0 0 3.14159"/>
-        <axis xyz="0 1 0"/>
+        <!-- Khung khớp đã quay pi quanh z nên trục 0 -1 0 (khung khớp) = +y của base_link, cùng chiều bánh trái:
+             vận tốc khớp dương ở cả hai bánh = robot tiến (giả định của gazebo_ros_diff_drive).
+             Bản gốc (0 1 0) làm bánh phải quay ngược -> lệnh tiến thành quay tại chỗ. -->
+        <axis xyz="0 -1 0"/>
     </joint>
     <link name="right_wheel">
@@ -154,5 +162,5 @@
             <origin xyz="0 0 0" rpy="0 0 0"/>
             <geometry>
-                <mesh filename="package://objectnav_sim_gazebo/meshes/hoverboard_motor_assembly.stl" scale="0.001 0.001 0.001"/>
+                <mesh filename="${mesh_uri}/hoverboard_motor_assembly.stl" scale="0.001 0.001 0.001"/>
             </geometry>
             <material name="blue"/>
@@ -178,5 +186,5 @@
             <origin xyz="0 0 0" rpy="0 0 0"/>
             <geometry>
-                <mesh filename="package://objectnav_sim_gazebo/meshes/caster_wheel.stl" scale="0.01 0.01 0.01"/>
+                <mesh filename="${mesh_uri}/caster_wheel.stl" scale="0.01 0.01 0.01"/>
             </geometry>
             <material name="black"/>
@@ -202,5 +210,5 @@
             <geometry>
                 <!-- <cylinder length="0.04" radius="0.038"/> -->
-                <mesh filename="package://objectnav_sim_gazebo/meshes/RPLiDAR_s2.stl" scale="0.001 0.001 0.001"/>
+                <mesh filename="${mesh_uri}/RPLiDAR_s2.stl" scale="0.001 0.001 0.001"/>
             </geometry>
             <material name="black"/>
@@ -210,5 +218,5 @@
             <geometry>
                 <cylinder length="0.04" radius="0.038"/>
-                <!-- <mesh filename="package://objectnav_sim_gazebo/meshes/RPLiDAR_s2.stl" scale="0.001 0.001 0.001"/> -->
+                <!-- <mesh filename="${mesh_uri}/RPLiDAR_s2.stl" scale="0.001 0.001 0.001"/> -->
             </geometry>
         </collision>
@@ -317,3 +325,78 @@
         <mu2>0.0</mu2>
     </gazebo>
+    <!-- LiDAR 2D: RPLIDAR S2/S2E theo thông số Slamtec — 0.05–30 m (phản xạ 90%), 10 Hz, 0.1125° (= 3200 tia/vòng,
+         32000 điểm/s), sai số ±30 mm, phân giải 13 mm. stddev 0.01 m là giả định (±30 mm ≈ 3σ), không có trong datasheet.
+         laser_frame quay pi như robot thật -> /scan cùng quy ước với sllidar_node (frame_id laser_frame).
+         Giảm lidar_samples (vd. 720) nếu real-time factor của Gazebo tụt. -->
+    <gazebo reference="laser_frame">
+        <sensor name="rplidar_s2" type="ray">
+            <always_on>true</always_on>
+            <visualize>false</visualize>
+            <update_rate>10</update_rate>
+            <ray>
+                <scan>
+                    <horizontal>
+                        <samples>${lidar_samples}</samples>
+                        <resolution>1</resolution>
+                        <min_angle>${-pi}</min_angle>
+                        <max_angle>${pi - 2*pi/float(lidar_samples)}</max_angle>
+                    </horizontal>
+                </scan>
+                <range>
+                    <min>0.05</min>
+                    <max>30.0</max>
+                    <resolution>0.013</resolution>
+                </range>
+                <noise>
+                    <type>gaussian</type>
+                    <mean>0.0</mean>
+                    <stddev>0.01</stddev>
+                </noise>
+            </ray>
+            <plugin name="rplidar_s2_plugin" filename="libgazebo_ros_ray_sensor.so">
+                <ros><remapping>~/out:=scan</remapping></ros>
+                <output_type>sensor_msgs/LaserScan</output_type>
+                <frame_name>laser_frame</frame_name>
+            </plugin>
+        </sensor>
+    </gazebo>
+    <!-- IMU: BNO055 trên robot thật publish /imu/data, frame imu_link, 100 Hz. IMU mô phỏng lý tưởng (không nhiễu). -->
+    <gazebo reference="imu_link">
+        <sensor name="bno055" type="imu">
+            <always_on>true</always_on>
+            <update_rate>100</update_rate>
+            <plugin name="bno055_plugin" filename="libgazebo_ros_imu_sensor.so">
+                <ros><remapping>~/out:=imu/data</remapping></ros>
+                <frame_name>imu_link</frame_name>
+                <initial_orientation_as_reference>false</initial_orientation_as_reference>
+            </plugin>
+        </sensor>
+    </gazebo>
+    <gazebo>
+        <!-- Dẫn động vi sai: /cmd_vel -> bánh, /odom từ encoder (odometry_source 0, có trượt như thật, không phải
+             ground truth). wheel_separation/diameter khớp wheel_odom_params.yaml (0.464 m, r = 0.084 m).
+             max_wheel_acceleration (m/s² tại vành bánh) = acc_lim_x của Nav2 (1.5); max_wheel_torque 20 N·m là giả định.
+             publish_odom_tf:=false khi chạy EKF (robot_localization) để tránh 2 nguồn TF odom->base_footprint. -->
+        <plugin name="diff_drive" filename="libgazebo_ros_diff_drive.so">
+            <update_rate>100</update_rate>
+            <left_joint>left_wheel_joint</left_joint>
+            <right_joint>right_wheel_joint</right_joint>
+            <wheel_separation>${2*wheel_offset_y}</wheel_separation>
+            <wheel_diameter>${2*wheel_radius}</wheel_diameter>
+            <max_wheel_torque>20</max_wheel_torque>
+            <max_wheel_acceleration>1.5</max_wheel_acceleration>
+            <publish_odom>true</publish_odom>
+            <publish_odom_tf>$(arg publish_odom_tf)</publish_odom_tf>
+            <publish_wheel_tf>false</publish_wheel_tf>
+            <odometry_frame>odom</odometry_frame>
+            <robot_base_frame>base_footprint</robot_base_frame>
+            <odometry_source>0</odometry_source>
+        </plugin>
+        <!-- /joint_states của 2 bánh -> robot_state_publisher phát TF base_link->left/right_wheel -->
+        <plugin name="joint_states" filename="libgazebo_ros_joint_state_publisher.so">
+            <update_rate>50</update_rate>
+            <joint_name>left_wheel_joint</joint_name>
+            <joint_name>right_wheel_joint</joint_name>
+        </plugin>
+    </gazebo>
 </robot>
